Commit message: update

File: src/robots/go2arm_description/urdf/go2arm_description.urdf (robot description, URDF)
Before this commit: robot go2arm_description, 39 links, 38 joints
Links:
- link FL_calf: geometry collision cylinder length=0.12 radius=0.012; visual mesh filename=package://go2arm_description/meshes/calf.dae
- link FL_foot: geometry collision sphere radius=0.022; visual mesh filename=package://go2arm_description/meshes/foot.dae
- link FL_hip: geometry collision cylinder length=0.04 radius=0.046; visual mesh filename=package://go2arm_description/meshes/hip.dae
- link FL_thigh: geometry collision box size=0.11 0.0245 0.034; visual mesh filename=package://go2arm_description/meshes/thigh.dae
- link FR_calf: geometry collision cylinder length=0.12 radius=0.013; visual mesh filename=package://go2arm_description/meshes/calf_mirror.dae
- link FR_foot: geometry collision sphere radius=0.022; visual mesh filename=package://go2arm_description/meshes/foot.dae
- link FR_hip: geometry collision cylinder length=0.04 radius=0.046; visual mesh filename=package://go2arm_description/meshes/hip.dae
- link FR_thigh: geometry collision box size=0.11 0.0245 0.034; visual mesh filename=package://go2arm_description/meshes/thigh_mirror.dae
- link RL_calf: geometry collision cylinder length=0.12 radius=0.013; visual mesh filename=package://go2arm_description/meshes/calf.dae
- link RL_foot: geometry collision sphere radius=0.022; visual mesh filename=package://go2arm_description/meshes/foot.dae
- link RL_hip: geometry collision cylinder length=0.04 radius=0.046; visual mesh filename=package://go2arm_description/meshes/hip.dae
- link RL_thigh: geometry collision box size=0.11 0.0245 0.034; visual mesh filename=package://go2arm_description/meshes/thigh.dae
- link RR_calf: geometry collision cylinder length=0.12 radius=0.013; visual mesh filename=package://go2arm_description/meshes/calf_mirror.dae
- link RR_foot: geometry collision sphere radius=0.022; visual mesh filename=package://go2arm_description/meshes/foot.dae
- link RR_hip: geometry collision cylinder length=0.04 radius=0.046; visual mesh filename=package://go2arm_description/meshes/hip.dae
- link RR_thigh: geometry collision box size=0.11 0.0245 0.034; visual mesh filename=package://go2arm_description/meshes/thigh_mirror.dae
- link base: geometry collision box size=0.3762 0.0935 0.114; visual mesh filename=package://go2arm_description/meshes/trunk.dae
- link base_link: geometry collision mesh filename=package://go2arm_description/meshes/base_link.dae; visual mesh filename=package://go2arm_description/meshes/base_link.dae
- link gripper_base: geometry collision mesh filename=package://go2arm_description/meshes/gripper_base.dae; visual mesh filename=package://go2arm_description/meshes/gripper_base.dae
- link link1: geometry collision mesh filename=package://go2arm_description/meshes/link1.dae; visual mesh filename=package://go2arm_description/meshes/link1.dae
- link link2: geometry collision mesh filename=package://go2arm_description/meshes/link2.dae; visual mesh filename=package://go2arm_description/meshes/link2.dae
- link link3: geometry collision mesh filename=package://go2arm_description/meshes/link3.dae; visual mesh filename=package://go2arm_description/meshes/link3.dae
- link link4: geometry collision mesh filename=package://go2arm_description/meshes/link4.dae; visual mesh filename=package://go2arm_description/meshes/link4.dae
- link link5: geometry collision mesh filename=package://go2arm_description/meshes/link5.dae; visual mesh filename=package://go2arm_description/meshes/link5.dae
- link link6: geometry collision mesh filename=package://go2arm_description/meshes/link6.dae; visual mesh filename=package://go2arm_description/meshes/link6.dae
- link link7: geometry collision mesh filename=package://go2arm_description/meshes/link7.dae; visual mesh filename=package://go2arm_description/meshes/link7.dae
- link link8: geometry collision mesh filename=package://go2arm_description/meshes/link8.dae; visual mesh filename=package://go2arm_description/meshes/link8.dae
